File: bus_board.kicad_pcb (KiCad board)
At the start: 2 copper layers, 483.9 x 39.4 mm, 67 parts, among them J1 Conn_02x05_Odd_Even, J10 Conn_02x05_Odd_Even, J11 Conn_02x08_Odd_Even, J12 Conn_02x08_Odd_Even, J13 Conn_02x08_Odd_Even, J14 Conn_02x08_Odd_Even, J15 Conn_02x08_Odd_Even, J16 Conn_02x08_Odd_Even, J17 P.C.B. mounting tabs, J18 Screw_Terminal_01x04, J19 Screw_Terminal_01x04, J2 Conn_02x05_Odd_Even, J20 P.C.B. mounting tabs, J21 P.C.B. mounting tabs, J22 P.C.B. mounting tabs, J23 P.C.B. mounting tabs, J24 P.C.B. mounting tabs, J25 P.C.B. mounting tabs, J26 P.C.B. mounting tabs, J27 Conn_02x03_Odd_Even, J28 Conn_02x05_Odd_Even, J29 Conn_02x05_Odd_Even, J3 Conn_02x05_Odd_Even, J30 Conn_02x05_Odd_Even, J31 Conn_02x05_Odd_Even, J32 Conn_02x05_Odd_Even, J33 Conn_02x05_Odd_Even, J34 Conn_02x05_Odd_Even, J35 Conn_02x05_Odd_Even, J36 Conn_02x05_Odd_Even, J37 Conn_02x05_Odd_Even, J38 Conn_02x08_Odd_Even, J39 Conn_02x08_Odd_Even, J4 Conn_02x05_Odd_Even, J40 Conn_02x08_Odd_Even, J41 Conn_02x08_Odd_Even, J42 Conn_02x08_Odd_Even, J43 Conn_02x08_Odd_Even, J44 Conn_02x03_Odd_Even, J5 Conn_02x05_Odd_Even, J6 Conn_02x05_Odd_Even, J7 Conn_02x05_Odd_Even, J8 Conn_02x05_Odd_Even, J9 Conn_02x05_Odd_Even

Commit message: Implement flood fills for power channels
Parts:
- moved C3 10.8 mm to (323.2, 213.7)
- moved C2 2.19 mm to (288.2, 203.9)
- moved C1 2.18 mm to (291.7, 209.2)
- moved R2 0.26 mm to (310.5, 218.2)
Routing:
- net -12V: track 630.2 -> 93.2 mm
- net +12V: track 583.3 -> 85.8 mm, vias 4 -> 2
- net +5V: track 546.3 -> 48.9 mm, vias 3 -> 2
- net CV: track 204.4 -> 220.1 mm
- net CV2: track 213.6 -> 224.4 mm
- net GATE: track 204.4 -> 210.4 mm
- net GND: vias 10 -> 11
- added copper zone on F.Cu, net +12V
- added copper zone on F.Cu, net +5V
- added copper zone on F.Cu, net -12V
Other:
- board size 483.9 x 39.4 mm -> 483.9 x 39.9 mm
